File: Hardware/ArduinoHotKey8/ArduinoHotKey8.sch (KiCad schematic (older format))
At the start: 1 part

Commit message: Compleded Circuit
Parts:
- added C1, C2, C3, C4, C5, C6, C7, C8: 100n, Capacitor_THT:C_Disc_D3.0mm_W1.6mm_P2.50mm, symbol Device:C
- added R1, R10, R11, R12, R13, R14, R15, R16, R2, R3, R4, R5, R6, R7, R8, R9: 10k, Resistor_THT:R_Axial_DIN0207_L6.3mm_D2.5mm_P10.16mm_Horizontal, symbol Device:R
- added SW0, SW1, SW2, SW3, SW4, SW5, SW6, SW7: SW_Push, Button_Switch_Keyboard:SW_Cherry_MX_1.00u_PCB, symbol Switch:SW_Push
- added SW_Reset1: SW_Push, Button_Switch_THT:SW_PUSH_6mm, symbol Switch:SW_Push
- B1: footprint ARDUINO_PRO_MINI -> SparkFun-KiCad-Libraries:ARDUINO_PRO_MINI
Connections:
- net BUTTON5: now reaches B1.10 (7)
- net BUTTON5: now also C6.1, R11.2
- net BUTTON6: now reaches B1.11 (8)
- net BUTTON6: now also C7.1, R13.2
- net BUTTON7: now reaches B1.12 (*9)
- net BUTTON7: now also C8.1, R15.2
- net VCC: now reaches B1.21 (VCC)
- net VCC: now also R10.1, R12.1, R14.1, R16.1, R2.1, R4.1, R6.1, R8.1
- net at B1.22 (RST): now also SW_Reset1.1
- net GND: now reaches B1.23 (GND)
- net GND: now also C1.2, C2.2, C3.2, C4.2, C5.2, C6.2, C7.2, C8.2, SW0.2, SW1.2, SW2.2, SW3.2, SW4.2, SW5.2, SW6.2, SW7.2, SW_Reset1.2
- net BUTTON0: now reaches B1.5 (2)
- net BUTTON0: now also C1.1, R1.2
- net BUTTON1: now reaches B1.6 (*3)
- net BUTTON1: now also C2.1, R3.2
- net BUTTON2: now reaches B1.7 (4)
- net BUTTON2: now also C3.1, R5.2
- net BUTTON3: now reaches B1.8 (*5)
- net BUTTON3: now also C4.1, R7.2
- net BUTTON4: now reaches B1.9 (*6)
- net BUTTON4: now also C5.1, R9.2
- new net: R1.1, R2.2, SW0.1
- new net: R3.1, R4.2, SW1.1
- new net: R5.1, R6.2, SW2.1
- new net: R7.1, R8.2, SW3.1
- new net: R10.2, R9.1, SW4.1
- new net: R11.1, R12.2, SW5.1
- new net: R13.1, R14.2, SW6.1
- new net: R15.1, R16.2, SW7.1
Other:
- moved on the sheet: B1

Commit message: First large PCB Design
Parts:
- removed B1: ARDUINO_PRO_MINI, SparkFun-KiCad-Libraries:ARDUINO_PRO_MINI, symbol SparkFun-Boards:ARDUINO_PRO_MINI
- added B1: SPARKFUN_PRO_MICRO, SparkFun-KiCad-Libraries:SPARKFUN_PRO_MICRO, symbol SparkFun-Boards:SPARKFUN_PRO_MICRO
- added H1, H2, H3, H4: MountingHole, MountingHole:MountingHole_3.2mm_M3, symbol Mechanical:MountingHole
Connections:
- net BUTTON0: now also B1.5 (2)
- net BUTTON1: now also B1.6 (*3)
- net BUTTON2: now also B1.7 (4)
- net BUTTON3: now also B1.8 (*5)
- net BUTTON4: now also B1.9 (*6)
- net BUTTON5: now also B1.10 (7)
- net BUTTON6: now also B1.11 (8)
- net BUTTON7: now also B1.12 (*9)
- net GND: now also B1.23 (GND)
- net VCC: now also B1.21 (VCC)
- net at SW_Reset1.1: now also B1.22 (RESET)
Changed lines of the file:
@@
 $EndDescr
-$Comp
-L SparkFun-Boards:ARDUINO_PRO_MINI B1
-U 1 1 5E9319F5
-P 2300 2050
-F 0 "B1" H 2300 3110 45  0000 C CNN
-F 1 "ARDUINO_PRO_MINI" H 2300 3026 45  0000 C CNN
-F 2 "SparkFun-KiCad-Libraries:ARDUINO_PRO_MINI" H 2300 3000 20  0001 C CNN
-F 3 "" H 2300 2050 50  0001 C CNN
-F 4 "XXX-00000" H 2300 2931 60  0000 C CNN "Feld4"
-	1    2300 2050
-	1    0    0    -1
-$EndComp
 $Comp
 L Switch:SW_Push SW0
@@
 	8650 5550 8650 5600
 Connection ~ 8450 5550
+$Comp
+L SparkFun-Boards:SPARKFUN_PRO_MICRO B1
+U 1 1 5E98BB34
+P 2300 1900
+F 0 "B1" H 2300 2810 45  0000 C CNN
+F 1 "SPARKFUN_PRO_MICRO" H 2300 2726 45  0000 C CNN
+F 2 "SparkFun-KiCad-Libraries:SPARKFUN_PRO_MICRO" H 2300 2700 20  0001 C CNN
+F 3 "" H 2300 1900 50  0001 C CNN
+F 4 "XXX-00000" H 2300 2631 60  0000 C CNN "Feld4"
+	1    2300 1900
+	1    0    0    -1
+$EndComp
+$Comp
+L Mechanical:MountingHole H1
+U 1 1 5E99EFEA
+P 5500 1500
+F 0 "H1" H 5600 1546 50  0000 L CNN
+F 1 "MountingHole" H 5600 1455 50  0000 L CNN
+F 2 "MountingHole:MountingHole_3.2mm_M3" H 5500 1500 50  0001 C CNN
+F 3 "~" H 5500 1500 50  0001 C CNN
+	1    5500 1500
+	1    0    0    -1
+$EndComp
+$Comp
+L Mechanical:MountingHole H2
+U 1 1 5E99FCF9
+P 5500 1750
+F 0 "H2" H 5600 1796 50  0000 L CNN
+F 1 "MountingHole" H 5600 1705 50  0000 L CNN
+F 2 "MountingHole:MountingHole_3.2mm_M3" H 5500 1750 50  0001 C CNN
+F 3 "~" H 5500 1750 50  0001 C CNN
+	1    5500 1750
+	1    0    0    -1
+$EndComp
+$Comp
+L Mechanical:MountingHole H3
+U 1 1 5E99FDBB
+P 5500 2000
+F 0 "H3" H 5600 2046 50  0000 L CNN
+F 1 "MountingHole" H 5600 1955 50  0000 L CNN
+F 2 "MountingHole:MountingHole_3.2mm_M3" H 5500 2000 50  0001 C CNN
+F 3 "~" H 5500 2000 50  0001 C CNN
+	1    5500 2000
+	1    0    0    -1
+$EndComp
+$Comp
+L Mechanical:MountingHole H4
+U 1 1 5E99FEBA
+P 5500 2250
+F 0 "H4" H 5600 2296 50  0000 L CNN
+F 1 "MountingHole" H 5600 2205 50  0000 L CNN
+F 2 "MountingHole:MountingHole_3.2mm_M3" H 5500 2250 50  0001 C CNN
+F 3 "~" H 5500 2250 50  0001 C CNN
+	1    5500 2250
+	1    0    0    -1
+$EndComp
 $EndSCHEMATC

Commit message: Added ISP Header
Added ISP Header and moved bulky parts to the back
Parts:
- added J1: AVR-ISP-6, Connector_IDC:IDC-Header_2x03_P2.54mm_Vertical, symbol Connector:AVR-ISP-6
Connections:
- net GND: now also J1.6 (GND)
- net VCC: now also J1.2 (VCC)
- net RST: now reaches B1.22 (RESET), SW_Reset1.1
- net RST: now also J1.5 (~RST)
- net MOSI: now reaches B1.14 (11(MOSI))
- net MOSI: now also J1.4 (MOSI)
- net MISO: now reaches B1.15 (12(MISO))
- net MISO: now also J1.1 (MISO)
- net SCK: now reaches B1.16 (13(SCK))
- net SCK: now also J1.3 (SCK)
Changed lines of the file:
@@
 	1    0    0    -1
 $EndComp
+$Comp
+L Connector:AVR-ISP-6 J1
+U 1 1 5E94559F
+P 4450 1600
+F 0 "J1" H 4171 1696 50  0000 R CNN
+F 1 "AVR-ISP-6" H 4171 1605 50  0000 R CNN
+F 2 "Connector_IDC:IDC-Header_2x03_P2.54mm_Vertical" V 4200 1650 50  0001 C CNN
+F 3 " ~" H 3175 1050 50  0001 C CNN
+	1    4450 1600
+	1    0    0    -1
+$EndComp
+$Comp
+L power:VCC #PWR0105
+U 1 1 5E9474AA
+P 4350 850
+F 0 "#PWR0105" H 4350 700 50  0001 C CNN
+F 1 "VCC" H 4367 1023 50  0000 C CNN
+F 2 "" H 4350 850 50  0001 C CNN
+F 3 "" H 4350 850 50  0001 C CNN
+	1    4350 850
+	1    0    0    -1
+$EndComp
+$Comp
+L power:GND #PWR0106
+U 1 1 5E947B34
+P 4350 2100
+F 0 "#PWR0106" H 4350 1850 50  0001 C CNN
+F 1 "GND" H 4355 1927 50  0000 C CNN
+F 2 "" H 4350 2100 50  0001 C CNN
+F 3 "" H 4350 2100 50  0001 C CNN
+	1    4350 2100
+	1    0    0    -1
+$EndComp
+Wire Wire Line
+	4350 2000 4350 2100
+Wire Wire Line
+	4350 850  4350 1100
+Wire Wire Line
+	4850 1400 5000 1400
+Wire Wire Line
+	4850 1500 5000 1500
+Wire Wire Line
+	4850 1600 5000 1600
+Wire Wire Line
+	4850 1700 5000 1700
+Text Label 5000 1400 0    50   ~ 0
+MISO
+Text Label 5000 1500 0    50   ~ 0
+MOSI
+Text Label 5000 1600 0    50   ~ 0
+SCK
+Text Label 5000 1700 0    50   ~ 0
+RST
+Text Label 2950 1550 0    50   ~ 0
+RST
+Wire Wire Line
+	2750 2150 2950 2150
+Wire Wire Line
+	2750 2250 2950 2250
+Wire Wire Line
+	2750 2350 2950 2350
+Text Label 2950 2250 0    50   ~ 0
+MISO
+Text Label 2950 2350 0    50   ~ 0
+MOSI
+Text Label 2950 2150 0    50   ~ 0
+SCK
 $EndSCHEMATC
